File: power_in.sch (KiCad schematic (older format))
At the start: 1 part

Commit message: addgit ignopre
Parts:
- removed J?: Conn_02x05_Row_Letter_Last, symbol Connector_Generic:Conn_02x05_Row_Letter_Last
- added J?: Conn_02x05_Top_Bottom, symbol Connector_Generic:Conn_02x05_Top_Bottom
Changed lines of the file:
@@
 $Descr A4 11693 8268
 encoding utf-8
-Sheet 4 4
+Sheet 5 6
 Title ""
 Date ""
@@
 $EndDescr
 $Comp
-L Connector_Generic:Conn_02x05_Row_Letter_Last J?
-U 1 1 5E302957
-P 2000 1800
-F 0 "J?" H 2050 2217 50  0000 C CNN
-F 1 "Conn_02x05_Row_Letter_Last" H 2050 2126 50  0000 C CNN
-F 2 "" H 2000 1800 50  0001 C CNN
-F 3 "~" H 2000 1800 50  0001 C CNN
-	1    2000 1800
+L Connector_Generic:Conn_02x05_Top_Bottom J?
+U 1 1 5E3153DB
+P 1150 1150
+AR Path="/5E3022E2/5E3153DB" Ref="J?"  Part="1"
+AR Path="/5E31859C/5E3153DB" Ref="J?"  Part="1"
+F 0 "J?" H 1200 1567 50  0000 C CNN
+F 1 "Conn_02x05_Top_Bottom" H 1200 1476 50  0000 C CNN
+F 2 "" H 1150 1150 50  0001 C CNN
+F 3 "~" H 1150 1150 50  0001 C CNN
+	1    1150 1150
 	1    0    0    -1
 $EndComp
