File: DAS_Power.sch (KiCad schematic (older format))
At the start: 0 parts

Commit message: addgit ignopre
Changed lines of the file:
@@
 $Descr A4 11693 8268
 encoding utf-8
-Sheet 1 4
+Sheet 1 6
 Title ""
 Date ""
@@
 Comment4 ""
 $EndDescr
-$Sheet
-S 1400 1900 500  150
-U 5E300FD5
-F0 "MCU" 50
-F1 "mcu.sch" 50
-$EndSheet
 $Sheet
 S 800  700  950  500
@@
 $EndSheet
 $Sheet
-S 2600 850  700  300
+S 800  2450 700  300
 U 5E3022E2
 F0 "Power Input" 50
 F1 "power_in.sch" 50
 $EndSheet
+$Sheet
+S 800  1800 700  300
+U 5E31859C
+F0 "Power Output" 50
+F1 "power_out.sch" 50
+$EndSheet
+$Sheet
+S 800  3150 1350 700
+U 5E31887A
+F0 "MCU" 50
+F1 "mcu.sch" 50
+$EndSheet
+$Sheet
+S 900  4200 500  150
+U 5E350920
+F0 "Fan Control" 50
+F1 "fan.sch" 50
+$EndSheet
 $EndSCHEMATC

Commit message: fac pmw v1
Changed lines of the file:
@@
 $EndSheet
 $Sheet
-S 900  4200 500  150
+S 800  4100 1350 600
 U 5E350920
 F0 "Fan Control" 50
 F1 "fan.sch" 50
+F2 "PWM_01" I L 800 4200 50
+F3 "PWM_02" I L 800 4300 50
+F4 "PWM_03" I L 800 4400 50
+F5 "PWM_04" I L 800 4500 50
+F6 "PWM_05" I L 800 4600 50
+F7 "FanSpeed01" O R 2150 4200 50
+F8 "FanSpeed02" O R 2150 4300 50
+F9 "FanSpeed03" O R 2150 4400 50
+F10 "FanSpeed04" O R 2150 4500 50
+F11 "FanSpeed05" O R 2150 4600 50
 $EndSheet
 $EndSCHEMATC
